Commit message: add mimic joints to exported URDF

File: onrobot_rg2_v2_description/urdf/onrobot_rg2_v2.xacro (robot description, xacro)
@@ -183,4 +183,6 @@
   <child link="finger1_inner_knuckle_link_1"/>
   <axis xyz="0.0 -0.0 -1.0"/>
+  <limit lower="-3.14" upper="3.14" effort="0.1" velocity="100" />
+  <mimic joint="finger1_joint" multiplier="1"/>
 </joint>
 <joint name="passive_finger1_tip_joint" type="continuous">
@@ -189,4 +191,6 @@
   <child link="finger1_tip_link_1"/>
   <axis xyz="-0.0 0.0 -1.0"/>
+  <limit lower="-3.14" upper="3.14" effort="0.1" velocity="100" />
+  <mimic joint="finger1_joint" multiplier="-1"/>
 </joint>
 <joint name="passive_finger2_joint" type="continuous">
@@ -195,4 +199,6 @@
   <child link="finger2_link_1"/>
   <axis xyz="-0.0 0.0 1.0"/>
+  <limit lower="-3.14" upper="3.14" effort="0.1" velocity="100" />
+  <mimic joint="finger1_joint" multiplier="1"/>
 </joint>
 <joint name="passive_finger2_innner_knuckle_joint" type="continuous">
@@ -201,4 +207,6 @@
   <child link="finger2_inner_knuckle_link_1"/>
   <axis xyz="-0.0 0.0 1.0"/>
+  <limit lower="-3.14" upper="3.14" effort="0.1" velocity="100" />
+  <mimic joint="passive_finger2_joint" multiplier="1"/>
 </joint>
 <joint name="passive_finger2_tip_joint" type="continuous">
@@ -207,4 +215,6 @@
   <child link="finger2_tip_link_1"/>
   <axis xyz="-0.0 -0.0 1.0"/>
+  <limit lower="-3.14" upper="3.14" effort="0.1" velocity="100" />
+  <mimic joint="passive_finger2_joint" multiplier="-1"/>
 </joint>
 </robot>
